File: CompaqSLT286-4MB.kicad_sch (KiCad schematic)
At the start: 26 parts, among them J116 Conn_02x30_Odd_Even, U1 74LS138, U2 74LS138, U3 IS61C5128AS-25TLI, U4 IS61C5128AS-25TLI, U5 IS61C5128AS-25TLI, U500 IS61C5128AS-25TLI, U501 IS61C5128AS-25TLI, U502 IS61C5128AS-25TLI, U503 IS61C5128AS-25TLI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

Commit message: fixed issue with detection pins; notes in schematics and updated production files
Parts:
- C1, C2, C500, C501, C502, C503, C504, C505, C506: value 100nF -> 47nF
- C508: value 100nF -> ?
- J116: value Conn_02x30_Odd_Even -> EDGE
- U1, U2: value 74LS138 -> 74AL138
- U7: value 74LS08 -> 74HC08
Connections:
- net +5V: now also C501.1, J116.49 (Pin_49); no longer C501.2, J116.45 (Pin_45)
- net GND: now also C501.2, J116.45 (Pin_45); no longer C501.1, J116.49 (Pin_49)
Other:
- note added: "Pins 45/49 are stick size detection! 45/49 H/L = 1MB 45/49 L/H = 4MB"
- moved on the sheet: J116, R1, R2, U1, U2
